File: examples/Teensy3ArtNetSACN2Universes_rdm/w550io_Teensy_DMX.brd (EAGLE design)
At the start: 98.7 x 64.8 mm, 33 parts, among them IC1 MAX481CPA, IC2 MAX481CPA

Commit message: Update RDM code and example
Parts:
- moved R4 5.24 mm to (19.1, 22.9)
Connections:
- net 3.3V: now also OK4.8, R4.2
- net 5VIN: no longer OK4.8, R4.1
- net GND: no longer OK4.3
- net N$1: now also OK4.3; no longer OK4.2
- net RX0: now also R4.1; no longer R4.2
- net VCC: now also OK4.2
Routing:
- net VCC: track 139.7 -> 86.4 mm
- net 5VIN: track 94.3 -> 65.1 mm
- net 3.3V: track 172.7 -> 195.6 mm
- net GND: track 183.4 -> 174.5 mm
- net TGND: track 190.8 -> 195.8 mm
- net RX0: track 29.2 -> 33.0 mm
- net N$1: track 58.4 -> 55.9 mm
Other:
- board text added: "copyright 2017 Claude Heintz Design"
- board text removed: "copyright 2016 Claude Heintz Design"
Changed lines of the file:
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@@
 <hole x="0" y="59.69" drill="2.2"/>
 <text x="35.56" y="60.96" size="1.27" layer="25" font="vector">http://lx.claudeheintzdesign.com/opensource.html</text>
-<text x="88.9" y="58.42" size="1.778" layer="25" font="vector" rot="R270">copyright 2016
+<text x="88.9" y="58.42" size="1.778" layer="25" font="vector" rot="R270">copyright 2017
 Claude Heintz Design</text>
 <text x="33.02" y="7.62" size="1.27" layer="25">Tx0</text>
@@
 <element name="R2" library="adafruit" package="0204/5" value="330Ω" x="34.29" y="29.21" rot="R180"/>
 <element name="R3" library="adafruit" package="0204/5" value="330Ω" x="41.91" y="29.21" rot="R180"/>
-<element name="R4" library="adafruit" package="0204/5" value="10k" x="24.13" y="24.13" rot="R180"/>
 <element name="IC1" library="maxim" package="DIL08" value="MAX481CPA" x="77.47" y="7.62" rot="R270">
 <attribute name="OC_FARNELL" value="unknown" x="77.47" y="7.62" size="1.778" layer="27" rot="R270" display="off"/>
@@
 <element name="C5" library="adafruit" package="B45181B" value="10uf" x="2.54" y="25.4"/>
 <element name="C6" library="adafruit" package="B45181B" value="10uf" x="2.54" y="21.59"/>
+<element name="R4" library="adafruit" package="0204/5" value="10k" x="19.05" y="22.86" rot="R180"/>
 </elements>
 <signals>
@@
 <wire x1="73.66" y1="54.61" x2="73.66" y2="39.37" width="0.4064" layer="16"/>
 <wire x1="60.96" y1="31.75" x2="60.96" y2="39.37" width="0.4064" layer="16"/>
-<wire x1="7.62" y1="19.05" x2="7.62" y2="22.86" width="0.4064" layer="16"/>
-<wire x1="7.62" y1="22.86" x2="24.13" y2="22.86" width="0.4064" layer="16"/>
-<wire x1="24.13" y1="22.86" x2="24.13" y2="19.05" width="0.4064" layer="16"/>
+<wire x1="7.62" y1="19.05" x2="7.62" y2="25.4" width="0.4064" layer="16"/>
+<wire x1="7.62" y1="25.4" x2="24.13" y2="25.4" width="0.4064" layer="16"/>
+<wire x1="24.13" y1="25.4" x2="24.13" y2="19.05" width="0.4064" layer="16"/>
 <contactref element="PWR" pad="2"/>
 <contactref element="C4" pad="1"/>
@@
 <wire x1="46.99" y1="19.05" x2="46.99" y2="17.78" width="0.4064" layer="16"/>
 <wire x1="46.99" y1="17.78" x2="34.29" y2="17.78" width="0.4064" layer="16"/>
-<wire x1="34.29" y1="17.78" x2="34.29" y2="19.05" width="0.4064" layer="16"/>
+<contactref element="OK4" pad="8"/>
+<wire x1="34.29" y1="19.05" x2="34.29" y2="17.78" width="0.4064" layer="16"/>
+<wire x1="34.29" y1="17.78" x2="16.51" y2="17.78" width="0.4064" layer="16"/>
+<wire x1="16.51" y1="17.78" x2="16.51" y2="19.05" width="0.4064" layer="16"/>
+<contactref element="R4" pad="2"/>
+<wire x1="16.51" y1="22.86" x2="16.51" y2="19.05" width="0.4064" layer="16"/>
 </signal>
 <signal name="RESET">
@@
 <contactref element="DC1" pad="2"/>
 <contactref element="TEENSY3R" pad="1"/>
-<contactref element="R4" pad="1"/>
 <wire x1="2.54" y1="49.53" x2="2.54" y2="21.59" width="0.4064" layer="16"/>
 <wire x1="2.54" y1="21.59" x2="2.54" y2="16.51" width="0.4064" layer="16"/>
@@
 <contactref element="C6" pad="+"/>
 <wire x1="7.62" y1="16.51" x2="16.51" y2="16.51" width="0" layer="19" extent="1-16"/>
-<wire x1="7.62" y1="16.51" x2="16.51" y2="16.51" width="0.4064" layer="16"/>
-<wire x1="16.51" y1="16.51" x2="26.67" y2="16.51" width="0.4064" layer="16"/>
-<wire x1="26.67" y1="16.51" x2="26.67" y2="24.13" width="0.4064" layer="16"/>
+<wire x1="16.51" y1="16.51" x2="26.67" y2="16.51" width="0" layer="19" extent="1-16"/>
 <wire x1="0" y1="25.4" x2="0" y2="21.59" width="0.4064" layer="16"/>
 <wire x1="0" y1="21.59" x2="2.54" y2="21.59" width="0.4064" layer="16"/>
 <wire x1="5.08" y1="52.07" x2="7.62" y2="53.34" width="0.4064" layer="16"/>
 <wire x1="7.62" y1="53.34" x2="8.89" y2="57.15" width="0.4064" layer="16"/>
-<contactref element="OK4" pad="8"/>
-<wire x1="16.51" y1="19.05" x2="16.51" y2="16.51" width="0.4064" layer="16"/>
-<wire x1="16.51" y1="16.51" x2="7.62" y2="16.51" width="0" layer="19" extent="1-16"/>
 </signal>
 <signal name="GND">
@@
 <contactref element="OK3" pad="5"/>
 <wire x1="54.61" y1="11.43" x2="54.61" y2="2.54" width="0.4064" layer="16"/>
-<contactref element="OK4" pad="3"/>
-<wire x1="21.59" y1="11.43" x2="21.59" y2="2.54" width="0.4064" layer="16"/>
 </signal>
 <signal name="VCC">
@@
 <wire x1="8.89" y1="7.62" x2="12.7" y2="7.62" width="0.4064" layer="16"/>
 <wire x1="73.66" y1="6.35" x2="73.66" y2="8.89" width="0.4064" layer="16"/>
-<wire x1="12.7" y1="7.62" x2="12.7" y2="13.97" width="0.4064" layer="16"/>
-<wire x1="12.7" y1="13.97" x2="21.59" y2="13.97" width="0.4064" layer="16"/>
-<wire x1="21.59" y1="13.97" x2="36.83" y2="13.97" width="0.4064" layer="16"/>
-<wire x1="36.83" y1="11.43" x2="36.83" y2="13.97" width="0.4064" layer="16"/>
-<wire x1="36.83" y1="13.97" x2="49.53" y2="13.97" width="0.4064" layer="16"/>
-<wire x1="49.53" y1="11.43" x2="49.53" y2="13.97" width="0.4064" layer="16"/>
-<wire x1="49.53" y1="13.97" x2="62.23" y2="13.97" width="0.4064" layer="16"/>
-<wire x1="62.23" y1="13.97" x2="62.23" y2="11.43" width="0.4064" layer="16"/>
 <wire x1="62.23" y1="11.43" x2="64.77" y2="11.43" width="0.4064" layer="16"/>
 <wire x1="64.77" y1="11.43" x2="64.77" y2="20.32" width="0.4064" layer="16"/>
@@
 <wire x1="77.47" y1="8.89" x2="77.47" y2="11.43" width="0.4064" layer="16"/>
 <wire x1="77.47" y1="11.43" x2="81.28" y2="11.43" width="0.4064" layer="16"/>
+<contactref element="OK4" pad="2"/>
+<wire x1="49.53" y1="11.43" x2="62.23" y2="11.43" width="0" layer="19" extent="1-1"/>
+<wire x1="36.83" y1="11.43" x2="49.53" y2="11.43" width="0" layer="19" extent="1-1"/>
+<wire x1="19.05" y1="11.43" x2="36.83" y2="11.43" width="0" layer="19" extent="1-1"/>
+<wire x1="12.7" y1="7.62" x2="19.05" y2="7.62" width="0.4064" layer="16"/>
+<wire x1="19.05" y1="7.62" x2="19.05" y2="11.43" width="0.4064" layer="16"/>
 </signal>
 <signal name="RX0">
 <contactref element="TEENSY3L" pad="2"/>
+<wire x1="7.62" y1="24.13" x2="7.62" y2="34.29" width="0.4064" layer="1"/>
+<wire x1="7.62" y1="24.13" x2="21.59" y2="24.13" width="0.4064" layer="1"/>
 <contactref element="OK4" pad="6"/>
-<wire x1="7.62" y1="24.13" x2="7.62" y2="34.29" width="0.4064" layer="1"/>
-<contactref element="R4" pad="2"/>
-<wire x1="21.59" y1="19.05" x2="21.59" y2="24.13" width="0.4064" layer="1"/>
-<wire x1="21.59" y1="24.13" x2="7.62" y2="24.13" width="0.4064" layer="1"/>
+<wire x1="21.59" y1="24.13" x2="21.59" y2="19.05" width="0.4064" layer="1"/>
+<contactref element="R4" pad="1"/>
+<wire x1="21.59" y1="22.86" x2="21.59" y2="19.05" width="0.4064" layer="16"/>
 </signal>
 <signal name="N$5">
@@
 </signal>
 <signal name="N$1">
+<contactref element="OK4" pad="3"/>
 <contactref element="R5" pad="1"/>
-<contactref element="OK4" pad="2"/>
 <wire x1="64.77" y1="24.13" x2="39.37" y2="24.13" width="0.4064" layer="1"/>
 <wire x1="39.37" y1="24.13" x2="39.37" y2="15.24" width="0.4064" layer="1"/>
-<wire x1="39.37" y1="15.24" x2="19.05" y2="15.24" width="0.4064" layer="1"/>
-<wire x1="19.05" y1="11.43" x2="19.05" y2="15.24" width="0.4064" layer="1"/>
+<wire x1="39.37" y1="15.24" x2="21.59" y2="15.24" width="0.4064" layer="1"/>
+<wire x1="21.59" y1="15.24" x2="21.59" y2="11.43" width="0.4064" layer="1"/>
+<wire x1="21.59" y1="11.43" x2="21.59" y2="11.43" width="0" layer="19" extent="1-16"/>
 </signal>
 </signals>
